File: Snake/Snake_hw/Snake.kicad_sch (KiCad schematic)
At the start: 82 parts, among them Q1 LED_RGB_CA, Q2 LED_RGB_CA, Q3 2N7002, Q4 IRLML6401, SW1 BUTTON, SW2 BUTTON, SW3 BUTTON, SW4 SWITCH

Commit message: + Snake layout done
Parts:
- removed ANT1: ANT_PCB_MONO_2PIN, Antennas:Locket5, symbol Antennas_kl:ANT_PCB_MONO_2PIN
- removed C4, C5: 18pF, Capacitors:CAP_0603, symbol Tittar_kl:C
- removed HOLE1, HOLE2, HOLE3, HOLE4: HOLE_METALLED, PCB:Hole2d2_out3d5mm, symbol pcb_details:HOLE_METALLED
- removed R3: 1k, Resistors:RES_0603, symbol Tittar_kl:R
- removed SW1, SW2: BUTTON, BtnsSwitches:BTN_IT1198, symbol Switches:BUTTON
- removed SW4: SWITCH, BtnsSwitches:SW_SS-1P2T_Housing, symbol Switches:SWITCH_1P2T_housing
- removed XL3: USB_MICRO, Connectors:USBmicro_MOLEX_1050170001, symbol Connectors_kl:USB_MINI_B
- removed XTAL1: 12MHz, Quartz:03225C4, symbol Tittar_kl:CRYSTAL_H
- added C31: 0.1u, Capacitors:CAP_0402, symbol Tittar_kl:C
- added F1: Fuse0R, Resistors:RES_0603_FUSE, symbol Tittar_kl:Fuse0R
- added Q5: IRLML9303, SOT:SOT23-3, symbol Transistors_kl:P_3PIN
- added Q6: BC848, SOT:SOT23-3, symbol Transistors_kl:NPN
- added R18, R20: 10k, Resistors:RES_0402_sm, symbol Tittar_kl:R
- added R19: 1M, Resistors:RES_0402_sm, symbol Tittar_kl:R
- added R21: 100k, Resistors:RES_0402_sm, symbol Tittar_kl:R
- added SW1, SW2: BUTTON, BtnsSwitches:BTN_4x4_SMD, symbol BtnsSwitches:BUTTON
- added XL3: USB_MICRO_6H, Connectors:USBmicro_MOLEX_1050170001, symbol Connectors_kl:USB_MICRO_6H
- added XL4, XL5: CONN_1, Connectors:PLS-1Square, symbol Connectors_kl:CONN_1
- B1: value BAT_HOLDER -> EEMB502030; footprint Installation:BATTERY_AAA_X2 -> Installation:EEMB502030; Price 5 -> (none); SolderPointsDIP 2 -> (none)
- C10, C11, C12, C13, C14, C15, C19, C20, C21, C22, C23, C24, C6, C7, C8: footprint Capacitors:CAP_0603 -> Capacitors:CAP_0402
- C16, C17, C25, C26, C27: footprint Capacitors:CAP_0603_Silks -> Capacitors:CAP_0402
- C18, C30: footprint Capacitors:CAP_0603 -> Capacitors:CAP_0603_Silks
- C9: value 10u -> 1u; footprint Capacitors:CAP_0603 -> Capacitors:CAP_0402
- Q4: value IRLML6401 -> IRLML9303; Price 5 -> (none)
- R1, R10, R11, R12, R13, R15, R16, R17, R2, R4, R5, R6, R7, R8, R9: footprint Resistors:RES_0603 -> Resistors:RES_0402_sm
- R14: footprint Resistors:RES_1206 -> Resistors:RES_0603
- SW3: Price (none) -> 1; SolderPoints (none) -> 4
Connections:
- net +BATT: now also F1.2, Q5.3 (D), R19.1, R21.1; no longer C29.2, C30.2, DA2.5 (BAT)
- net 5V_USB: now also Q5.1 (G), XL3.1 (UVcc); no longer Q4.1 (G)
- net ANT2: now also XL4.1 (P1)
- net BAT_IN: now also C29.2, C30.2, DA2.5 (BAT), Q4.2 (S), F1.1, R18.1
- net BTN1: now also SW1.2
- net BTN2: now also SW2.2
- net GND: now also C31.2, Q6.2 (E), XL3.4 (UID), XL3.5 (UGND), XL5.1 (P1)
- net PwrMCU: now also SW1.1, SW2.1; no longer SW3.2
- net PwrUnst: now also Q5.2 (S); no longer Q4.2 (S)
- net USB_DM: now also XL3.2 (D-)
- net USB_DP: now also XL3.3 (D+)
- net BTN3: no longer names the net of DD1.13 (ADC8/SAI1MCLKA/T15C2/T2C4/LP1RX/RX2/PA3)
- net BTN3: no longer SW3.1
- new net: Q6.3 (C), R18.2, R20.2
- new net: C31.1, R19.2, SW3.2
- new net: Q6.1 (B), R21.2
- new net PWRBTN1: Q4.1 (G), R20.1, SW3.1
- no-connect marks 14 -> 18
Other:
- moved on the sheet: C26, C27, C30, D1, DA1, R17
