File: Snake/Snake_hw/Snake.kicad_pcb (KiCad board)
At the start: 4 copper layers, 46.9 x 30.9 mm, 82 parts, among them Q1 LED_RGB_CA, Q2 LED_RGB_CA, Q3 2N7002, Q4 IRLML9303, Q5 IRLML9303, Q6 BC848, SW1 BUTTON, SW2 BUTTON, SW3 BUTTON

Commit message: + Snake sent to production + Knout layout done
Parts:
- moved Logo1 17.8 mm to (139.2, 108.2)
- moved L3 14.1 mm to (139.6, 105.2)
- moved TP4 1.15 mm to (128.4, 92.5)
- moved R5 1.10 mm to (131.0, 115.7)
- moved R6 1.10 mm to (131.0, 116.7)
- moved R7 1.10 mm to (131.0, 117.7)
- moved R11 0.16 mm to (138.4, 114.9)
- moved R12 0.16 mm to (138.4, 112.9)
- moved DA2 0.10 mm to (117.8, 100.3)
- turned R17 to 0 degrees
- turned R9 to 180 degrees
Routing:
- net GND: track 0.00 -> 209.4 mm, vias 0 -> 77
- net PwrMCU: track 0.00 -> 72.0 mm, vias 0 -> 6
- net /PWRBTN1: track 0.00 -> 48.2 mm, vias 0 -> 1
- net +BATT: track 0.00 -> 47.8 mm
- net /5V_USB: track 0.00 -> 44.0 mm, vias 0 -> 4
- net VCC: track 0.00 -> 43.9 mm, vias 0 -> 6
- net +3v3: track 0.00 -> 39.5 mm, vias 0 -> 4
- net /GREEN_LED: track 0.00 -> 33.1 mm, vias 0 -> 3
- net /BLUE_LED: track 0.00 -> 32.5 mm, vias 0 -> 3
- net /RED_LED: track 0.00 -> 30.4 mm, vias 0 -> 3
- net /BTN1: track 0.00 -> 29.0 mm, vias 0 -> 4
- net /BAT_IN: track 0.00 -> 25.1 mm, vias 0 -> 3
- net /USB_DM: track 0.00 -> 23.9 mm
- net /USB_DP: track 0.00 -> 23.8 mm
- net /CC_CS: track 0.00 -> 23.0 mm, vias 0 -> 3
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- added copper zone on B.Cu, net GND
- added copper zone on F.Cu, net GND
- added copper zone on In1.Cu, net GND
- added copper zone on In2.Cu, net GND
Other:
- board text added: "Ostranna"
- board text added: "Snake v1"
