File: Knout/Knout_hw/Knout.kicad_sch (KiCad schematic)
At the start: 88 parts, among them Q1 IRF9317, Q2 2N7002, Q3 2N7002, Q4 IRLML9303, Q6 BC848, Q7 IRLML6401, SW1 BUTTON_H

Commit message: + Snake fw started
Parts:
- Logo1: footprint Pictures:Ostranna_12d7_10d1 -> Pictures:Ostranna_8x8
Changed lines of the file:
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@@
       (effects (font (size 1.524 1.524)))
     )
-    (property "Footprint" "Pictures:Ostranna_12d7_10d1" (id 2) (at 394.97 233.68 0)
+    (property "Footprint" "Pictures:Ostranna_8x8" (id 2) (at 394.97 233.68 0)
       (effects (font (size 1.524 1.524)) hide)
     )
@@
     )
     (path "/56931bf1-2ca5-4096-af7f-97ec749bdf9d"
-      (reference "Logo1") (unit 1) (value "Logo") (footprint "Pictures:Ostranna_12d7_10d1")
+      (reference "Logo1") (unit 1) (value "Logo") (footprint "Pictures:Ostranna_8x8")
     )
     (path "/75be1d4e-bab7-48a1-9f80-1b1cac95b915"
